Commit message: reconfig model joint relation

File: spot_description/urdf/accessories.urdf.xacro (robot description, xacro)
@@ -3,15 +3,16 @@
   <xacro:if value="$(optenv SPOT_PACK 0)">
     <joint name="pack_mount_joint" type="fixed">
-      <parent link="base_link"/>
+      <parent link="body"/>
       <child link="pack_mount"/>
-      <origin xyz="-0.019986 0 0.093662" rpy="0 0 0"/>
+      <origin xyz="-0.13 0 0.12" rpy="0 0 0"/>
     </joint>
     <link name="pack_mount">
       <visual>
         <geometry>
-          <mesh filename="package://spot_description/meshes/pack_top.dae"/>
+          <box size="0.21 0.15 0.075"/>
+          <!-- <mesh filename="package://spot_description/meshes/pack_top.dae"/> -->
         </geometry>
       </visual>
-      <visual>
+      <!-- <visual>
         <geometry>
           <mesh filename="package://spot_description/meshes/pack_body.dae"/>
@@ -22,5 +23,5 @@
           <mesh filename="package://spot_description/meshes/pack_body.dae"/>
         </geometry>
-      </collision>
+      </collision> -->
     </link>
   </xacro:if>
@@ -29,8 +30,8 @@
       <parent link="pack_mount"/>
       <child link="lidar_mount"/>
-      <origin xyz="0.015 0 0.149285" rpy="0 0 0"/>
+      <origin xyz="-0.11 0 0.05" rpy="0 0 0"/>
     </joint>
     <link name="lidar_mount">
-      <visual>
+      <!-- <visual>
         <geometry>
           <mesh filename="package://spot_description/meshes/lidar_mount.dae"/>
@@ -41,5 +42,5 @@
           <mesh filename="package://spot_description/meshes/lidar_mount_collision.stl"/>
         </geometry>
-      </collision>
+      </collision> -->
     </link>
     <xacro:if value="$(optenv SPOT_VELODYNE 0)">

File: spot_description/urdf/spot_arm.xacro (robot description, xacro)
@@ -66,10 +66,10 @@
 <link name="finger">
   <inertial>
-    <origin rpy="0 0 0" xyz="0.8635899028063472 0.09862056591557622 0.00850232975194119"/>
+    <origin rpy="0.3 0 0" xyz="0.0 0.05 0.0"/>
     <mass value="1.71236178687828"/>
     <inertia ixx="0.002129" ixy="0.0" ixz="-0.0" iyy="0.001681" iyz="0.000162" izz="0.003403"/>
   </inertial>
   <visual>
-    <origin rpy="0 0 0" xyz="0.87709 -0.823505 -0.0185"/>
+    <origin rpy="0.3 0 0" xyz="0.0 0.05 -0.0"/>
     <geometry>
       <mesh filename="package://spot_description/meshes/arm/finger.stl" scale="0.001 0.001 0.001"/>
@@ -78,5 +78,5 @@
   </visual>
   <collision>
-    <origin rpy="0 0 0" xyz="0.87709 -0.823505 -0.0185"/>
+    <origin rpy="0.3 0 0" xyz="0.0 0.05 -0.0"/>
     <geometry>
       <mesh filename="package://spot_description/meshes/arm/finger.stl" scale="0.001 0.001 0.001"/>
@@ -165,8 +165,8 @@
 </link>
 <joint name="base_arm_joint" type="fixed">
-        <origin xyz="0.29 0 0.08" rpy="0 0 0" />
-        <parent link="body" />
-        <child link="base_arm_link" />
-    </joint>
+  <origin xyz="0.29 0 0.08" rpy="0 0 0" />
+  <parent link="body" />
+  <child link="base_arm_link" />
+</joint>
 <joint name="arm_joint1" type="revolute">
   <origin rpy="0 0 0" xyz="0.0 0.0 0.065"/>
@@ -177,8 +177,8 @@
 </joint>
 <joint name="arm_joint2" type="revolute">
-  <origin rpy="0 0 0" xyz="0.015 0.0 0.05"/>
+  <origin rpy="3.1415 0 1.57" xyz="0.015 0.0 0.05"/>
   <parent link="link1"/>
   <child link="link2"/>
-  <axis xyz="-1.0 0.0 0.0"/>
+  <axis xyz="1.0 0.0 0.0"/>
   <limit effort="100" lower="-3.665191" upper="0.0" velocity="100"/>
 </joint>
@@ -212,5 +212,5 @@
 </joint>
 <joint name="arm_gripper" type="revolute">
-  <origin rpy="0 0 0" xyz="-0.86859 0.043915 -0.029"/>
+  <origin rpy="0 0 0" xyz="-0.0 0.06 0.0"/>
   <parent link="gripper"/>
   <child link="finger"/>

Commit message: update urdf & control profile

File: spot_description/urdf/accessories.urdf.xacro (robot description, xacro)
@@ -47,5 +47,5 @@
       <!-- Use the Velodyne macro for the actual sensor -->
       <xacro:include filename="$(find velodyne_description)/urdf/VLP-16.urdf.xacro" />
-      <xacro:VLP-16 parent="lidar_mount">
+      <xacro:VLP-16 parent="velodyne_cage">
         <origin xyz="$(optenv SPOT_VELODYNE_XYZ 0 0 0)" rpy="$(optenv SPOT_VELODYNE_RPY 0 0 0)" />
       </xacro:VLP-16>
@@ -57,5 +57,4 @@
           </geometry>
           <origin xyz="0 0 0" rpy="0 0 0" />
-          <material name="black" />
         </visual>
         <collision>

Commit message: add microstrain imu & edit urdf & tune controller

File: spot_description/urdf/accessories.urdf.xacro (robot description, xacro)
@@ -75,3 +75,24 @@
     <xacro:include filename="$(find spot_description)/urdf/spot_arm.xacro" />
   </xacro:if>
+  <xacro:if value="$(optenv SPOT_IMU 0)">
+    <link name="imu">
+      <visual>
+          <geometry>
+            <box size="0.033 0.0245 0.0127"/>
+          </geometry>
+          <origin xyz="0 0 0" rpy="0 0 0" />
+        </visual>
+        <collision>
+          <geometry>
+            <box size="0.033 0.0245 0.0127"/>
+          </geometry>
+          <origin xyz="0 0 0" rpy="0 0 0" />
+        </collision>
+    </link>
+    <joint name="imu_joint" type="fixed">
+        <parent link="velodyne_cage" />
+        <child link="imu" />
+        <origin xyz="0 0 0.08" rpy="3.1415 0 0" />
+      </joint>
+  </xacro:if>
 </robot>

Commit message: update IMU position (move below Lidar)

File: spot_description/urdf/accessories.urdf.xacro (robot description, xacro)
@@ -93,5 +93,5 @@
         <parent link="velodyne_cage" />
         <child link="imu" />
-        <origin xyz="0 0 0.08" rpy="3.1415 0 0" />
+        <origin xyz="-0.04 0 -0.01" rpy="0 0 3.1415" />
       </joint>
   </xacro:if>

Commit message: update urdf

File: spot_description/urdf/accessories.urdf.xacro (robot description, xacro)
@@ -30,5 +30,5 @@
       <parent link="pack_mount"/>
       <child link="lidar_mount"/>
-      <origin xyz="-0.11 0 0.05" rpy="0 0 0"/>
+      <origin xyz="-0.05 0 0.26" rpy="0 0 0"/>
     </joint>
     <link name="lidar_mount">
